File: hardware/kicad/Emiuet_plate/Emiuet_plate.kicad_pcb (KiCad board)
At the start: 2 copper layers, 297 x 102.4 mm, 102 parts

Commit message: Fix Kicad Data
Other:
- board text added: "5V"
- board text added: "DATA"
- board text added: "MIDI"
- board text added: "ON OFF"
- board text added: "↔"
