File: hardware/kicad/Emiuet.kicad_pcb (KiCad board)
At the start: 2 copper layers, 297 x 102.4 mm, 264 parts, among them J1 USB_C_Receptacle_USB2.0_16P, J2 USB_C_Receptacle_USB2.0_16P, J3 AudioJack3, J4 Conn_01x02_Pin, Q1 S9013 J3, SW1 SW_Slide_DPDT, SW1_0 Switch_SW_Push, SW1_1 Switch_SW_Push, SW1_10 Switch_SW_Push, SW1_11 Switch_SW_Push, SW1_12 Switch_SW_Push, SW1_2 Switch_SW_Push, SW1_3 Switch_SW_Push, SW1_4 Switch_SW_Push, SW1_5 Switch_SW_Push, SW1_6 Switch_SW_Push, SW1_7 Switch_SW_Push, SW1_8 Switch_SW_Push, SW1_9 Switch_SW_Push, SW2 SW_SPST, SW2_0 Switch_SW_Push, SW2_1 Switch_SW_Push, SW2_10 Switch_SW_Push, SW2_11 Switch_SW_Push, SW2_12 Switch_SW_Push, SW2_2 Switch_SW_Push, SW2_3 Switch_SW_Push, SW2_4 Switch_SW_Push, SW2_5 Switch_SW_Push, SW2_6 Switch_SW_Push, SW2_7 Switch_SW_Push, SW2_8 Switch_SW_Push, SW2_9 Switch_SW_Push, SW3 SW_SPST, SW3_0 Switch_SW_Push, SW3_1 Switch_SW_Push, SW3_10 Switch_SW_Push, SW3_11 Switch_SW_Push, SW3_12 Switch_SW_Push, SW3_2 Switch_SW_Push, SW3_3 Switch_SW_Push, SW3_4 Switch_SW_Push, SW3_5 Switch_SW_Push, SW3_6 Switch_SW_Push, SW3_7 Switch_SW_Push, SW3_8 Switch_SW_Push, SW3_9 Switch_SW_Push, SW4 SW_SPST, SW4_0 Switch_SW_Push, SW4_1 Switch_SW_Push, SW4_10 Switch_SW_Push, SW4_11 Switch_SW_Push, SW4_12 Switch_SW_Push, SW4_2 Switch_SW_Push, SW4_3 Switch_SW_Push, SW4_4 Switch_SW_Push, SW4_5 Switch_SW_Push, SW4_6 Switch_SW_Push, SW4_7 Switch_SW_Push, SW4_8 Switch_SW_Push, SW4_9 Switch_SW_Push, SW5_0 Switch_SW_Push, SW5_1 Switch_SW_Push, SW5_10 Switch_SW_Push, SW5_11 Switch_SW_Push, SW5_12 Switch_SW_Push, SW5_2 Switch_SW_Push, SW5_3 Switch_SW_Push, SW5_4 Switch_SW_Push, SW5_5 Switch_SW_Push, SW5_6 Switch_SW_Push, SW5_7 Switch_SW_Push, SW5_8 Switch_SW_Push, SW5_9 Switch_SW_Push, SW6_0 Switch_SW_Push, SW6_1 Switch_SW_Push, SW6_10 Switch_SW_Push, SW6_11 Switch_SW_Push, SW6_12 Switch_SW_Push, SW6_2 Switch_SW_Push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

Commit message: Fix Kicad Data
Parts:
- removed JP1: Jumper_2_Bridged, TestPoint:TestPoint_2Pads_Pitch2.54mm_Drill0.8mm
- removed JP3: Jumper_2_Bridged, Jumper:SolderJumper-2_P1.3mm_Bridged_RoundedPad1.0x1.5mm
- BT1: footprint EUB_Passives:Battery Cell 800mah bis -> EUB_Passives:Battery Cell 800mah nobis; moved to B.Cu
- moved J4 36.2 mm to (87.6, 77.1)
- moved TH1 13.5 mm to (81.8, 95.4), turned to 90 degrees
- moved C23 3.69 mm to (337.7, 138.8), turned to 90 degrees
- moved BT1 3.37 mm to (67.0, 95.8), turned to 90 degrees
Connections:
- C21 pad 1: Net-(JP1-B) -> USB1_VBUS
- C22 pad 1: Net-(JP1-B) -> USB1_VBUS
- TH1 pad 1: Net-(JP3-B) -> Net-(U7-TS)
- U7 pad 1: Net-(JP3-A) -> Net-(U7-TS)
- U7 pad 13: Net-(JP1-B) -> USB1_VBUS
Routing:
- net Net-(JP3-B): track 288.0 -> 0.00 mm, vias 6 -> 0
- net Net-(U7-TS): track 0.00 -> 284.1 mm, vias 0 -> 8
- net SDA: track 331.8 -> 347.0 mm
- net SCL: track 331.4 -> 345.4 mm, vias 7 -> 6
- net Net-(JP3-A): track 9.78 -> 0.00 mm, vias 2 -> 0
- net Net-(JP1-B): track 8.11 -> 0.00 mm
- net Net-(J4-Pin_1): track 404.8 -> 402.2 mm
- net USB1_VBUS: track 73.1 -> 75.6 mm
- net Frt12: track 324.9 -> 326.9 mm
- net SYS: track 67.7 -> 66.2 mm
- net Net-(U1-EN): track 5.06 -> 4.94 mm, vias 2 -> 0
- net GNDD: vias 394 -> 390
- net GNDA: vias 327 -> 338

Commit message: KiCad REV-B Design
Parts:
- added C31: 1μ, EUB_Passives:C_0603_1608Metric_noSilks, F.Cu at (339.9, 131.8)
- added R6: 10k, EUB_Passives:R_0603_1608Metric_noSilks, F.Cu at (338.3, 113.0)
- added R7: JP_TX0, EUB_Passives:R_0603_1608Metric_noSilks, F.Cu at (333.1, 44.2)
- added R8: JP_RX0, EUB_Passives:R_0603_1608Metric_noSilks, F.Cu at (84.6, 135.9)
- added SW5: SW_SPST, Button_Switch_SMD:SW_SPST_TS-1088-xR020, F.Cu at (338.9, 135.5)
- added TP1: TestPoint, TestPoint:TestPoint_Pad_D1.0mm, F.Cu at (338.9, 111.2)
- added TP2: TestPoint, TestPoint:TestPoint_Pad_D1.0mm, F.Cu at (338.8, 109.1)
- added TP3: TestPoint, TestPoint:TestPoint_Pad_D1.0mm, F.Cu at (333.2, 130.6)
- added TP4: TestPoint, TestPoint:TestPoint_Pad_D1.0mm, F.Cu at (330.4, 133.5)
- added TP5: TestPoint, TestPoint:TestPoint_Pad_D1.0mm, F.Cu at (331.8, 132.1)
- moved R5 5.96 mm to (333.2, 100.6), turned to 0 degrees
- moved C20 3.73 mm to (78.9, 135.8)
- moved R26 3.64 mm to (325.7, 135.0)
- moved R25 3.64 mm to (324.2, 135.0)
- moved G*** 3.17 mm to (69.4, 59.0)
- moved C18 2.69 mm to (75.9, 135.8)
- moved C1 1.40 mm to (335.0, 133.0)
- moved C21 0.42 mm to (334.2, 134.7)
- moved R1 0.36 mm to (336.5, 131.5)
Connections:
- U1 pad 39: TXD -> Net-(U1-TXD0)
- U1 pad 4: unconnected-(U1-IO0-Pad4) -> BOOT
- U1 pad 40: SW_LEFT -> Net-(U1-RXD0)
Routing:
- net Net-(U1-RXD0): track 0.00 -> 253.7 mm
- net SW_LEFT: track 262.5 -> 12.2 mm
- net Net-(U1-TXD0): track 0.00 -> 98.9 mm, vias 0 -> 6
- net TXD: track 94.0 -> 3.88 mm, vias 6 -> 0
- net Net-(SW5-A): track 4.94 -> 12.1 mm
- net Net-(D3-A): track 9.32 -> 3.37 mm
- net +3V3: track 451.0 -> 456.5 mm
- net PGOOD: track 26.6 -> 28.6 mm
- net Frt0: track 134.2 -> 135.9 mm
- net Frt1: track 158.6 -> 160.2 mm
- net BOOT: track 0.00 -> 1.48 mm
- net Net-(U7-TS): track 284.1 -> 285.3 mm
- net SW_CENTER: track 274.9 -> 273.9 mm
- net USB1_VBUS: track 75.6 -> 74.7 mm
- net SYS: track 66.2 -> 67.0 mm
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Other:
- board text added: "BOOT"
- board text added: "GND"
- board text added: "JP RX0"
- board text added: "JP TX0"
- board text added: "LED R"
- board text added: "RST"
- board text added: "RX"
- board text added: "Rev B - Jan 2026"
- board text added: "TX"
- board text added: "USB1/5V"
- board text added: "USB2/DATA"
- board text removed: "LED R1k-"
- board text removed: "Rev A - Dec 2025"
- board text removed: "TS"
- board text removed: "USB1/POW"
- board text removed: "USB1_VBUS"
- board text removed: "USB2/COM"
