File: hardware/kicad/Emiuet.kicad_pcb (KiCad board)
At the start: 2 copper layers, 297 x 102.4 mm, 275 parts, among them J1 USB_C_Receptacle_USB2.0_16P, J2 USB_C_Receptacle_USB2.0_16P, J3 AudioJack3, J4 Conn_01x02_Pin, Q1 S9013 J3, SW1 SW_Slide_DPDT, SW1_0 Switch_SW_Push, SW1_1 Switch_SW_Push, SW1_10 Switch_SW_Push, SW1_11 Switch_SW_Push, SW1_12 Switch_SW_Push, SW1_2 Switch_SW_Push, SW1_3 Switch_SW_Push, SW1_4 Switch_SW_Push, SW1_5 Switch_SW_Push, SW1_6 Switch_SW_Push, SW1_7 Switch_SW_Push, SW1_8 Switch_SW_Push, SW1_9 Switch_SW_Push, SW2 SW_SPST, SW2_0 Switch_SW_Push, SW2_1 Switch_SW_Push, SW2_10 Switch_SW_Push, SW2_11 Switch_SW_Push, SW2_12 Switch_SW_Push, SW2_2 Switch_SW_Push, SW2_3 Switch_SW_Push, SW2_4 Switch_SW_Push, SW2_5 Switch_SW_Push, SW2_6 Switch_SW_Push, SW2_7 Switch_SW_Push, SW2_8 Switch_SW_Push, SW2_9 Switch_SW_Push, SW3 SW_SPST, SW3_0 Switch_SW_Push, SW3_1 Switch_SW_Push, SW3_10 Switch_SW_Push, SW3_11 Switch_SW_Push, SW3_12 Switch_SW_Push, SW3_2 Switch_SW_Push, SW3_3 Switch_SW_Push, SW3_4 Switch_SW_Push, SW3_5 Switch_SW_Push, SW3_6 Switch_SW_Push, SW3_7 Switch_SW_Push, SW3_8 Switch_SW_Push, SW3_9 Switch_SW_Push, SW4 SW_SPST, SW4_0 Switch_SW_Push, SW4_1 Switch_SW_Push, SW4_10 Switch_SW_Push, SW4_11 Switch_SW_Push, SW4_12 Switch_SW_Push, SW4_2 Switch_SW_Push, SW4_3 Switch_SW_Push, SW4_4 Switch_SW_Push, SW4_5 Switch_SW_Push, SW4_6 Switch_SW_Push, SW4_7 Switch_SW_Push, SW4_8 Switch_SW_Push, SW4_9 Switch_SW_Push, SW5 SW_SPST, SW5_0 Switch_SW_Push, SW5_1 Switch_SW_Push, SW5_10 Switch_SW_Push, SW5_11 Switch_SW_Push, SW5_12 Switch_SW_Push, SW5_2 Switch_SW_Push, SW5_3 Switch_SW_Push, SW5_4 Switch_SW_Push, SW5_5 Switch_SW_Push, SW5_6 Switch_SW_Push, SW5_7 Switch_SW_Push, SW5_8 Switch_SW_Push, SW5_9 Switch_SW_Push, SW6 SW_SPST, SW6_0 Switch_SW_Push, SW6_1 Switch_SW_Push, SW6_10 Switch_SW_Push, SW6_11 Switch_SW_Push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

Commit message: BOOTスイッチ修正
Parts:
- moved R6 2.70 mm to (338.9, 110.3), turned to -90 degrees
Connections:
- SW6 pad 1: +3V3 -> BOOT
Routing:
- net BOOT: track 1.48 -> 9.18 mm, vias 0 -> 2
- net +3V3: track 468.0 -> 462.2 mm
Other:
- board text added: "lroevie Saidai M gray Ai Muhao Tsrulino Nakahiro zakk rairai Orange Cat UdenIrphus"
- board text removed: "lroevie Saidai M gray Ai Muhao Tsrulino Nakahiro zakk rairai Orange Cat"
