File: hardware/kicad/Emiuet.kicad_sch (KiCad schematic)
At the start: 272 parts, among them J1 USB_C_Receptacle_USB2.0_16P, J2 USB_C_Receptacle_USB2.0_16P, J3 AudioJack3, J4 Conn_01x02_Pin, Q1 S9013 J3, SW1 SW_Slide_DPDT, SW1_0 Switch_SW_Push, SW1_1 Switch_SW_Push, SW1_10 Switch_SW_Push, SW1_11 Switch_SW_Push, SW1_12 Switch_SW_Push, SW1_2 Switch_SW_Push, SW1_3 Switch_SW_Push, SW1_4 Switch_SW_Push, SW1_5 Switch_SW_Push, SW1_6 Switch_SW_Push, SW1_7 Switch_SW_Push, SW1_8 Switch_SW_Push, SW1_9 Switch_SW_Push, SW2 SW_SPST, SW2_0 Switch_SW_Push, SW2_1 Switch_SW_Push, SW2_10 Switch_SW_Push, SW2_11 Switch_SW_Push, SW2_12 Switch_SW_Push, SW2_2 Switch_SW_Push, SW2_3 Switch_SW_Push, SW2_4 Switch_SW_Push, SW2_5 Switch_SW_Push, SW2_6 Switch_SW_Push, SW2_7 Switch_SW_Push, SW2_8 Switch_SW_Push, SW2_9 Switch_SW_Push, SW3 SW_SPST, SW3_0 Switch_SW_Push, SW3_1 Switch_SW_Push, SW3_10 Switch_SW_Push, SW3_11 Switch_SW_Push, SW3_12 Switch_SW_Push, SW3_2 Switch_SW_Push, SW3_3 Switch_SW_Push, SW3_4 Switch_SW_Push, SW3_5 Switch_SW_Push, SW3_6 Switch_SW_Push, SW3_7 Switch_SW_Push, SW3_8 Switch_SW_Push, SW3_9 Switch_SW_Push, SW4 SW_SPST, SW4_0 Switch_SW_Push, SW4_1 Switch_SW_Push, SW4_10 Switch_SW_Push, SW4_11 Switch_SW_Push, SW4_12 Switch_SW_Push, SW4_2 Switch_SW_Push, SW4_3 Switch_SW_Push, SW4_4 Switch_SW_Push, SW4_5 Switch_SW_Push, SW4_6 Switch_SW_Push, SW4_7 Switch_SW_Push, SW4_8 Switch_SW_Push, SW4_9 Switch_SW_Push, SW5 SW_SPST, SW5_0 Switch_SW_Push, SW5_1 Switch_SW_Push, SW5_10 Switch_SW_Push, SW5_11 Switch_SW_Push, SW5_12 Switch_SW_Push, SW5_2 Switch_SW_Push, SW5_3 Switch_SW_Push, SW5_4 Switch_SW_Push, SW5_5 Switch_SW_Push, SW5_6 Switch_SW_Push, SW5_7 Switch_SW_Push, SW5_8 Switch_SW_Push, SW5_9 Switch_SW_Push, SW6 SW_SPST, SW6_0 Switch_SW_Push, SW6_1 Switch_SW_Push, SW6_10 Switch_SW_Push, SW6_11 Switch_SW_Push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

Commit message: Rev.BをUSB給電RGB構成へ更新
- 単一USB-C Device/UFP給電へ回路方針を変更（内蔵電池・充電・PowerPath・boost・Host VBUS経路を撤去）
- TUSB320を固定UFPとしI2C status読出しのみに限定
- SK6812 MINI-E x78のRGB chain、AHCT level shift、RMT/DMA rendererを追加
- USB MIDI + HID Keyboard composite、TRS MIDI IN/OUTを整理
- firmware: led_control/led_renderer/midi_input/usb_power/tusb320/board_i2c を追加
- KiCad: Rev.A schematicをEmiuet_RevA.kicad_schへ退避し、Rev.B初期schematicたたき台を追加
- docs: README/decisions/pinout-v3/keyboard-mode をRev.B仕様へ更新、Rev.A資料をdocs/history/へ移動
Parts:
- removed BT1: 800mAh, EUB_Passives:Battery Cell 800mah nobis, symbol EUB_Passives:BatteryCell_800mAh
- removed Brd2: waveshare0.96inch, EUB_SSD1306:9E6018AD, symbol SSD1306-128x64_OLED:waveshare0.96inch
- removed C1, C12, C31: 1μ, EUB_Passives:C_0603_1608Metric_noSilks, symbol Device:C_Small
- removed C10: 33p, EUB_Passives:C_0603_1608Metric_noSilks, symbol Device:C_Small
- removed C11, C13, C15, C16, C17, C18, C19, C20, C22, C25, C27, C30, C5, C8, C9: 100n, EUB_Passives:C_0603_1608Metric_noSilks, symbol Device:C_Small
- removed C14, C21, C23, C24, C28, C29, C3, C4, C6, C7: 22μ, EUB_Passives:C_0603_1608Metric_noSilks, symbol Device:C_Small
- removed C2: 10μ, EUB_Passives:C_0603_1608Metric_noSilks, symbol Device:C_Small
- removed C26: Byp or Bulk xμ_10μ, EUB_Passives:C_0603_1608Metric_noSilks, symbol Device:C_Small
- removed D1: SMF5V0A, Eminuet Library:D_SOD-123F_noSilk, symbol Diode:SMF5V0A
- removed D1_0, D1_1, D1_10, D1_11, D1_12, D1_2, D1_3, D1_4, D1_5, D1_6, D1_7, D1_8, D1_9, D2_0, D2_1, D2_10, D2_11, D2_12, D2_2, D2_3, D2_4, D2_5, D2_6, D2_7, D2_8, D2_9, D3_0, D3_1, D3_10, D3_11, D3_12, D3_2, D3_3, D3_4, D3_5, D3_6, D3_7, D3_8, D3_9, D4_0, D4_1, D4_10, D4_11, D4_12, D4_2, D4_3, D4_4, D4_5, D4_6, D4_7, D4_8, D4_9, D5_0, D5_1, D5_10, D5_11, D5_12, D5_2, D5_3, D5_4, D5_5, D5_6, D5_7, D5_8, D5_9, D6_0, D6_1, D6_10, D6_11, D6_12, D6_2, D6_3, D6_4, D6_5, D6_6, D6_7, D6_8, D6_9: 1N4148, EUB_Passives:D_SOD-123_no silks, symbol Device:D_Small
- removed D3: LED B, Eminuet Library:LED_D5.0mm THT Turn_noSilk, symbol Device:LED
- removed F1, F2: MF-MSMF110-2, Eminuet Library:Fuse_1812_4532Metric_noSilk, symbol Device:Polyfuse_Small
- removed FB1, FB2: FerriteBead_Small, Eminuet Library:L_0805_2012Metric_noSilk, symbol Device:FerriteBead_Small
- removed H_Center1, H_Center2, H_Center3, H_Center4, H_Center5, H_Center6, H_Center7, H_Center8, H_Left1, H_Left2, H_Left3, H_Left4, H_Right1, H_Right2, H_Right3, H_Right4: MountingHole, EUB_MountingHole:MountingHole_2.2mm_M2_jlcpcb, symbol Mechanical:MountingHole
- removed J2: USB_C_Receptacle_USB2.0_16P, Eminuet Library:USB_C_Receptacle_G-Switch_GT-USB-7010ASV_noSilk, symbol Connector:USB_C_Receptacle_USB2.0_16P
- removed J4: Conn_01x02_Pin, EUB_Passives:JST_PH_B2B-PH-SM4-TB_1x02-1MP_P2.00mm_Vertical_right+, symbol Connector:Conn_01x02_Pin
- removed L1: DLW21SN900SQ2L, EUB_KeySwitches:L_CommonModeChoke_Coilcraft_0603USB_noSilk, symbol Filter:Choke_Wurth_WE-CNSW_744232090
- removed L2: 4.7μ, EUB_Passives:L_TDK_VLS6045EX_VLS6045AF_noSilk, symbol Device:L_Small
- removed NT2: NetTie_2, NetTie:NetTie-2_SMD_Pad0.5mm, symbol Device:NetTie_2
- removed Q1: S9013 J3, Eminuet Library:SOT-23_noSilk, symbol Transistor_BJT:BC817
- removed R1, R10, R25, R26, R6: 10k, EUB_Passives:R_0603_1608Metric_noSilks, symbol Device:R_Small_US
- removed R11: 900k, EUB_Passives:R_0603_1608Metric_noSilks, symbol Device:R_Small_US
- removed R12, R17, R18: 4.7k, EUB_Passives:R_0603_1608Metric_noSilks, symbol Device:R_Small_US
- removed R13: 887k, EUB_Passives:R_0603_1608Metric_noSilks, symbol Device:R_Small_US
- removed R14: 120k, EUB_Passives:R_0603_1608Metric_noSilks, symbol Device:R_Small_US
- removed R15: 200k, Eminuet Library:R_1206_3216Metric_noSilk, symbol Device:R_Small_US
- removed R16: 200k, EUB_Passives:R_0603_1608Metric_noSilks, symbol Device:R_Small_US
- removed R19, R20, R21: 100, EUB_Passives:R_0603_1608Metric_noSilks, symbol Device:R_Small_US
- removed R2, R3: 5.1k, EUB_Passives:R_0603_1608Metric_noSilks, symbol Device:R_Small_US
- removed R22: 1.18k, EUB_Passives:R_0603_1608Metric_noSilks, symbol Device:R_Small_US
- removed R23: 4.12k, EUB_Passives:R_0603_1608Metric_noSilks, symbol Device:R_Small_US
- removed R24: 1.13k, EUB_Passives:R_0603_1608Metric_noSilks, symbol Device:R_Small_US
- removed R27: 560k, Resistor_THT:R_Axial_DIN0204_L3.6mm_D1.6mm_P7.62mm_Horizontal, symbol Device:R_Small_US
- removed R28: 1k, EUB_Passives:R_0603_1608Metric_noSilks, symbol Device:R_Small_US
- removed R29: 220k, EUB_Passives:R_0603_1608Metric_noSilks, symbol Device:R_Small_US
- removed R30: 100k, EUB_Passives:R_0603_1608Metric_noSilks, symbol Device:R_Small_US
- removed R4, R9: 220, EUB_Passives:R_0603_1608Metric_noSilks, symbol Device:R_Small_US
- removed R5: 1k, Resistor_THT:R_Axial_DIN0204_L3.6mm_D1.6mm_P7.62mm_Horizontal, symbol Device:R_Small_US
- removed R7, R8: 470, EUB_Passives:R_0603_1608Metric_noSilks, symbol Device:R_Small_US
- removed RV1, RV2, RV3: 10k, EUB_Passives:Potentiometer_Slider_AliExpress_10k_35mm, symbol Device:R_Potentiometer_Trim
- removed SW1: SW_Slide_DPDT, EUB_Passives:SW_SK22D02_DPDT_Angled, symbol Switch:SW_Slide_DPDT
- removed SW1_0, SW1_1, SW1_10, SW1_11, SW1_12, SW1_2, SW1_3, SW1_4, SW1_5, SW1_6, SW1_7, SW1_8, SW1_9, SW2_0, SW2_1, SW2_10, SW2_11, SW2_12, SW2_2, SW2_3, SW2_4, SW2_5, SW2_6, SW2_7, SW2_8, SW2_9, SW3_0, SW3_1, SW3_10, SW3_11, SW3_12, SW3_2, SW3_3, SW3_4, SW3_5, SW3_6, SW3_7, SW3_8, SW3_9, SW4_0, SW4_1, SW4_10, SW4_11, SW4_12, SW4_2, SW4_3, SW4_4, SW4_5, SW4_6, SW4_7, SW4_8, SW4_9, SW5_0, SW5_1, SW5_10, SW5_11, SW5_12, SW5_2, SW5_3, SW5_4, SW5_5, SW5_6, SW5_7, SW5_8, SW5_9, SW6_0, SW6_1, SW6_10, SW6_11, SW6_12, SW6_2, SW6_3, SW6_4, SW6_5, SW6_6, SW6_7, SW6_8, SW6_9: Switch_SW_Push, EUB_KeySwitches:SW_Hotswap_Kailh_Choc_noD_reflect, symbol sweepv2-cache:Switch_SW_Push
- removed SW2: SW_SPST, EUB_Passives:Akidsuki_WhiteCircleTactileSwitch, symbol Switch:SW_SPST
- removed SW3, SW4: SW_SPST, EUB_Passives:SW_PUSH_6mm_H9.5mm_DTS65, symbol Switch:SW_SPST
- removed SW5, SW6: SW_SPST, Button_Switch_SMD:SW_SPST_TS-1088-xR020, symbol Switch:SW_SPST
- removed SW7, SW8: SW_SPDT, Button_Switch_SMD:SW_SPDT_Shouhan_MSK12C02, symbol Switch:SW_SPDT
- removed TH1: Thermistor, EUB_Passives:R_0603_1608Metric_noSilks, symbol Device:Thermistor
- removed TP1, TP3, TP4, TP5: TestPoint, TestPoint:TestPoint_Pad_D1.0mm, symbol Connector:TestPoint
- removed U2: TPD2EUSB30ADRTR, Eminuet Library:Texas_DRT-3_noSilk, symbol Power_Protection:TPD2EUSB30
- removed U3: LM66100DCK, Eminuet Library:SOT-363_SC-70-6_noSilk, symbol Power_Management:LM66100DCK
- removed U4: AP7333-33SAG-7, Eminuet Library:SOT-23_noSilk, symbol Regulator_Linear:AP7381-28SA-7
- removed U5: TUSB320LAIRWBR, Eminuet Library:Texas_X2QFN-12_1.6x1.6mm_P0.4mm_noSilk, symbol Interface_USB:TUSB320
- removed U6: TPS61023DRLR, Eminuet Library:SOT-563_noSilk, symbol EUB_Passives:TPS61023DRLR
- removed U7: BQ24074RGT, Eminuet Library:BQ24074_QFN-16_3x3mm_withThermalVia_noSilk, symbol Battery_Management:BQ24074RGT
- added C1: 680uF TBD, symbol Device:C_Polarized
- added D1, D10, D11, D12, D13, D14, D15, D16, D17, D18, D19, D2, D20, D21, D22, D23, D24, D25, D26, D27, D28, D29, D3, D30, D31, D32, D33, D34, D35, D36, D37, D38, D39, D4, D40, D41, D42, D43, D44, D45, D46, D47, D48, D49, D5, D50, D51, D52, D53, D54, D55, D56, D57, D58, D59, D6, D60, D61, D62, D63, D64, D65, D66, D67, D68, D69, D7, D70, D71, D72, D73, D74, D75, D76, D77, D78, D8, D9: SK6812MINI-E, LED_SMD:LED_SK6812MINI-E_3.2x2.8mm_P1.5mm_ReverseMount, symbol LED:SK6812MINI-E
- added J2: TRS MIDI OUT Type-A, symbol Connector_Audio:AudioJack3
- added U2: TUSB320LAI, symbol Interface_USB:TUSB320
- added U3: 3V3_REGULATOR_TBD_600mA, symbol Regulator_Linear:AP2112K-3.3
- added U4: SN74AHCT1G125, symbol 74xGxx:74AHCT1G125
- added U5: MIDI_IN_OPTO_TBD, symbol Isolator:6N138
- J1: value USB_C_Receptacle_USB2.0_16P -> USB-C Device/UFP; footprint Eminuet Library:USB_C_Receptacle_G-Switch_GT-USB-7010ASV_noSilk -> (none)
- J3: value AudioJack3 -> TRS MIDI IN Type-A; footprint EUB_Passives:Jack_3.5mm_KoreanHropartsElec_PJ-313D-4A_Horizontal -> (none)
- U1: value ESP32-S3-MINI-1 -> ESP32-S3-MINI-1-N4R2; footprint Eminuet Library:ESP32-S2-MINI-1_thermalVia_noSilk -> (none)
Connections:
- net D+ is gone; now on net USB_D+: U1.24 (USB_D+)
- net D- is gone; now on net USB_D-: U1.23 (USB_D-)
- net Frt7 is gone; now on net SW_LEFT: U1.27 (IO47)
- net +3V3: now also U2.12 (VDD)
- net SW_CENTER: now also U1.37 (IO41); no longer U1.36 (IO40)
- net SW_RIGHT: now also U1.38 (IO42); no longer U1.35 (IO39)
- net USB_VBUS: now reaches J1.A4 (VBUS), J1.A9 (VBUS), J1.B4 (VBUS), J1.B9 (VBUS)
- net EN_RESET: now reaches U1.45 (EN)
- net CC1: now reaches J1.A5 (CC1)
- net CC1: now also U2.1 (CC1)
- net USB_D+: now reaches J1.A6 (D+)
- net USB_D+: now also J1.B6 (D+)
- net USB_D-: now reaches J1.A7 (D-)
- net USB_D-: now also J1.B7 (D-)
- net CC2: now reaches J1.B5 (CC2)
- net CC2: now also U2.2 (CC2)
- net STRAP_GPIO3_SPARE: now reaches U1.7 (IO3)
- net BAT_VSENSE renamed COL6
- net BOOT renamed BOOT_GPIO0
- net CHG renamed PILOT_LED
- net FLASH_RX renamed MIDI_IN_RX_GPIO44
- net FLASH_TX renamed MIDI_OUT_TX_GPIO43
- net Frt0: no longer names the net of U1.44 (IO46)
- net Frt1: no longer names the net of U1.41 (IO45)
- net Frt10 renamed COL3
- net Frt11 renamed COL2
- net Frt12 renamed COL1
- net Frt2 renamed COL11
- net Frt3 renamed COL12
- net Frt4 renamed TUSB_INT_N
- net TUSB_INT_N: now also U2.6 (~{INT}/OUT3)
- net Frt5 renamed COL10
- net Frt6 renamed COL9
- net Frt8 renamed COL8
- net Frt9 renamed COL4
- net GNDD renamed GND
- net GND: now also D1.1 (VSS), D10.1 (VSS), D11.1 (VSS), D12.1 (VSS), D13.1 (VSS), D14.1 (VSS), D15.1 (VSS), D16.1 (VSS), D17.1 (VSS), D18.1 (VSS), D19.1 (VSS), D2.1 (VSS), D20.1 (VSS), D21.1 (VSS), D22.1 (VSS), D23.1 (VSS), D24.1 (VSS), D25.1 (VSS), D26.1 (VSS), D27.1 (VSS), D28.1 (VSS), D29.1 (VSS), D3.1 (VSS), D30.1 (VSS), D31.1 (VSS), D32.1 (VSS), D33.1 (VSS), D34.1 (VSS), D35.1 (VSS), D36.1 (VSS), D37.1 (VSS), D38.1 (VSS), D39.1 (VSS), D4.1 (VSS), D40.1 (VSS), D41.1 (VSS), D42.1 (VSS), D43.1 (VSS), D44.1 (VSS), D45.1 (VSS), D46.1 (VSS), D47.1 (VSS), D48.1 (VSS), D49.1 (VSS), D5.1 (VSS), D50.1 (VSS), D51.1 (VSS), D52.1 (VSS), D53.1 (VSS), D54.1 (VSS), D55.1 (VSS), D56.1 (VSS), D57.1 (VSS), D58.1 (VSS), D59.1 (VSS), D6.1 (VSS), D60.1 (VSS), D61.1 (VSS), D62.1 (VSS), D63.1 (VSS), D64.1 (VSS), D65.1 (VSS), D66.1 (VSS), D67.1 (VSS), D68.1 (VSS), D69.1 (VSS), D7.1 (VSS), D70.1 (VSS), D71.1 (VSS), D72.1 (VSS), D73.1 (VSS), D74.1 (VSS), D75.1 (VSS), D76.1 (VSS), D77.1 (VSS), D78.1 (VSS), D8.1 (VSS), D9.1 (VSS), U2.10 (GND); no longer J1.S1 (SHIELD), J3.S
- net LED renamed ROW1
- net PGOOD renamed RGB_DATA_3V3
- net RGB_DATA_3V3: now also U4.2
- net SCL renamed COL5
- net SDA renamed COL7
- net SLDR1 renamed SLIDER_VEL
- net SLDR2 renamed SLIDER_MOD
- net SLDR3 renamed SLIDER_PB
- net Str1 renamed ROW0
- net Str2 renamed ROW2
- net Str3 renamed ROW3
- net Str4 renamed ROW4
- net Str5 renamed COL0
- net Str6 renamed ROW5
- new net: D1.4 (DOUT), D2.2 (DIN)
- new net: D2.4 (DOUT), D3.2 (DIN)
- new net: D3.4 (DOUT), D4.2 (DIN)
- new net: D4.4 (DOUT), D5.2 (DIN)
- new net: D5.4 (DOUT), D6.2 (DIN)
- new net: D6.4 (DOUT), D7.2 (DIN)
- new net: D7.4 (DOUT), D8.2 (DIN)
- new net: D8.4 (DOUT), D9.2 (DIN)
- new net: D10.2 (DIN), D9.4 (DOUT)
- new net: D10.4 (DOUT), D11.2 (DIN)
- new net: D11.4 (DOUT), D12.2 (DIN)
- new net: D12.4 (DOUT), D13.2 (DIN)
- new net: D13.4 (DOUT), D14.2 (DIN)
- new net: D14.4 (DOUT), D15.2 (DIN)
- new net: D15.4 (DOUT), D16.2 (DIN)
- new net: D16.4 (DOUT), D17.2 (DIN)
- new net: D17.4 (DOUT), D18.2 (DIN)
- new net: D18.4 (DOUT), D19.2 (DIN)
- new net: D19.4 (DOUT), D20.2 (DIN)
- new net: D20.4 (DOUT), D21.2 (DIN)
- new net: D21.4 (DOUT), D22.2 (DIN)
- new net: D22.4 (DOUT), D23.2 (DIN)
- new net: D23.4 (DOUT), D24.2 (DIN)
- new net: D24.4 (DOUT), D25.2 (DIN)
- new net: D25.4 (DOUT), D26.2 (DIN)
- new net: D26.4 (DOUT), D27.2 (DIN)
- new net: D27.4 (DOUT), D28.2 (DIN)
- new net: D28.4 (DOUT), D29.2 (DIN)
- new net: D29.4 (DOUT), D30.2 (DIN)
- new net: D30.4 (DOUT), D31.2 (DIN)
- new net: D31.4 (DOUT), D32.2 (DIN)
- new net: D32.4 (DOUT), D33.2 (DIN)
- new net: D33.4 (DOUT), D34.2 (DIN)
- new net: D34.4 (DOUT), D35.2 (DIN)
- new net: D35.4 (DOUT), D36.2 (DIN)
- new net: D36.4 (DOUT), D37.2 (DIN)
- new net: D37.4 (DOUT), D38.2 (DIN)
- new net: D38.4 (DOUT), D39.2 (DIN)
- new net: D39.4 (DOUT), D40.2 (DIN)
- new net: D40.4 (DOUT), D41.2 (DIN)
- new net: D41.4 (DOUT), D42.2 (DIN)
- new net: D42.4 (DOUT), D43.2 (DIN)
- new net: D43.4 (DOUT), D44.2 (DIN)
- new net: D44.4 (DOUT), D45.2 (DIN)
- new net: D45.4 (DOUT), D46.2 (DIN)
- new net: D46.4 (DOUT), D47.2 (DIN)
- new net: D47.4 (DOUT), D48.2 (DIN)
- new net: D48.4 (DOUT), D49.2 (DIN)
- new net: D49.4 (DOUT), D50.2 (DIN)
- new net: D50.4 (DOUT), D51.2 (DIN)
- new net: D51.4 (DOUT), D52.2 (DIN)
- new net: D52.4 (DOUT), D53.2 (DIN)
- new net: D53.4 (DOUT), D54.2 (DIN)
- new net: D54.4 (DOUT), D55.2 (DIN)
- new net: D55.4 (DOUT), D56.2 (DIN)
- new net: D56.4 (DOUT), D57.2 (DIN)
- new net: D57.4 (DOUT), D58.2 (DIN)
- new net: D58.4 (DOUT), D59.2 (DIN)
- new net: D59.4 (DOUT), D60.2 (DIN)
- new net: D60.4 (DOUT), D61.2 (DIN)
- new net: D61.4 (DOUT), D62.2 (DIN)
- new net: D62.4 (DOUT), D63.2 (DIN)
- new net: D63.4 (DOUT), D64.2 (DIN)
- new net: D64.4 (DOUT), D65.2 (DIN)
- new net: D65.4 (DOUT), D66.2 (DIN)
- new net: D66.4 (DOUT), D67.2 (DIN)
- new net: D67.4 (DOUT), D68.2 (DIN)
- new net: D68.4 (DOUT), D69.2 (DIN)
- new net: D69.4 (DOUT), D70.2 (DIN)
- new net: D70.4 (DOUT), D71.2 (DIN)
- new net: D71.4 (DOUT), D72.2 (DIN)
- new net: D72.4 (DOUT), D73.2 (DIN)
- new net: D73.4 (DOUT), D74.2 (DIN)
- new net: D74.4 (DOUT), D75.2 (DIN)
- new net: D75.4 (DOUT), D76.2 (DIN)
- new net: D76.4 (DOUT), D77.2 (DIN)
- new net: D77.4 (DOUT), D78.2 (DIN)
- new net +5V_LED: D1.3 (VDD), D10.3 (VDD), D11.3 (VDD), D12.3 (VDD), D13.3 (VDD), D14.3 (VDD), D15.3 (VDD), D16.3 (VDD), D17.3 (VDD), D18.3 (VDD), D19.3 (VDD), D2.3 (VDD), D20.3 (VDD), D21.3 (VDD), D22.3 (VDD), D23.3 (VDD), D24.3 (VDD), D25.3 (VDD), D26.3 (VDD), D27.3 (VDD), D28.3 (VDD), D29.3 (VDD), D3.3 (VDD), D30.3 (VDD), D31.3 (VDD), D32.3 (VDD), D33.3 (VDD), D34.3 (VDD), D35.3 (VDD), D36.3 (VDD), D37.3 (VDD), D38.3 (VDD), D39.3 (VDD), D4.3 (VDD), D40.3 (VDD), D41.3 (VDD), D42.3 (VDD), D43.3 (VDD), D44.3 (VDD), D45.3 (VDD), D46.3 (VDD), D47.3 (VDD), D48.3 (VDD), D49.3 (VDD), D5.3 (VDD), D50.3 (VDD), D51.3 (VDD), D52.3 (VDD), D53.3 (VDD), D54.3 (VDD), D55.3 (VDD), D56.3 (VDD), D57.3 (VDD), D58.3 (VDD), D59.3 (VDD), D6.3 (VDD), D60.3 (VDD), D61.3 (VDD), D62.3 (VDD), D63.3 (VDD), D64.3 (VDD), D65.3 (VDD), D66.3 (VDD), D67.3 (VDD), D68.3 (VDD), D69.3 (VDD), D7.3 (VDD), D70.3 (VDD), D71.3 (VDD), D72.3 (VDD), D73.3 (VDD), D74.3 (VDD), D75.3 (VDD), D76.3 (VDD), D77.3 (VDD), D78.3 (VDD), D8.3 (VDD), D9.3 (VDD)
- new net GND_ADDR_0x60: U2.5 (ADDR)
- new net GND_EN_N: U2.11 (~{EN})
- new net GND_PORT_UFP: U2.3 (PORT)
- new net I2C_SCL: U1.36 (IO40), U2.8 (SCL/OUT2)
- new net I2C_SDA: U1.35 (IO39), U2.7 (SDA/OUT1)
- new net RGB_DATA_5V_AFTER_68R: D1.2 (DIN)
- new net RGB_DATA_OUT_TEST: D78.4 (DOUT)
- new net SHIELD_RC_GND_TBD: J1.SH (SHIELD)
- new net VBUS_DET_900K: U2.4 (VBUS_DET)
- no-connect marks 20 -> 0
Other:
- note added: "3 ADC sliders + 3 buttons + OLED on shared I2C"
- note added: "6x13 matrix (78 Choc + diode + hotswap); rows/columns above are routed as grouped buses in PCB redesign"
- note added: "Bulk 470-1000uF candidate; input protection/inrush and regulator choice remain validation items"
- note added: "CURRENT: single USB-C / fixed UFP / no battery / no Host VBUS"
- note added: "D1..Dn chain order is serpentine; firmware logical 6x13 coordinates are mapped separately"
- note added: "Emiuet Rev.B USB-powered controller"
- note added: "GPIO allocation is defined in docs/pinout-v3.md; GPIO0/3/45/46 reserved for boot/strapping"
- note added: "OUT: MIDI 3.3V electrical spec buffer/current limiting. IN: optocoupler + reverse diode; no jack signal/shield DC path to GND"
- note added: "SK6812 MINI-E DATA CHAIN: 78 pixels; every pixel has local 100nF (candidate), power is parallel"
- note added: "U2 fixed UFP: PORT=L, ADDR=L (0x60), EN_N=L, VBUS_DET via 900k; no DRP/source control"
- note added: "U4 VCC=+5V_LED, OE=L; 68R candidate between buffer and D1"
- note added: "VBUS -> TVS + 1.5A-rated fuse/eFuse -> +5V_LED; USB D+/D- -> low-C ESD -> GPIO20/19"
- note removed: "3.3 V 低ドロップアウトレギュレータ（LDO）"
- note removed: "Analog GND"
- note removed: "ESD保護素子(USB端子から最短)"
- note removed: "FLAS用UART確保"
- note removed: "TRS MIDI TypeA 信号線を要確認"
- note removed: "USB2 保護"
- note removed: "USBのCCライン制御"
- note removed: "コモンドチョーク"
- note removed: "データ/電源両用USB USB2"
- note removed: "バッテリー充電管理と電源の切り替え"
- note removed: "右側インターフェイス"
- note removed: "同じ長さにする"
- note removed: "安定3.3V"
- note removed: "安定5V"
- note removed: "左側インターフェイス"
- note removed: "昇圧型DC/DCコンバータ"
- note removed: "理想ダイオード／逆流防止スイッチ"
- note removed: "電源トグル/充電監視LED"
- note removed: "電源供給専用USB USB1"
- company: (none) -> Emnyeca
- title: (none) -> Emiuet Rev.B USB-powered controller

Commit message: Rev.BのCC検出と送信taskを整備しレビュー指摘を修正
Parts:
- removed U2: TUSB320LAI, symbol Interface_USB:TUSB320
- added C2: 1u, Capacitor_SMD:C_0603_1608Metric, symbol Device:C
- added C3: 10u, Capacitor_SMD:C_0603_1608Metric, symbol Device:C
- added C4, C5, C6, C9: 100n, Capacitor_SMD:C_0603_1608Metric, symbol Device:C
- added C7, C8: 10n, Capacitor_SMD:C_0603_1608Metric, symbol Device:C
- added J4: Waveshare 0.96inch OLED (C), Eminuet Library:Waveshare_OLED_0.96in_C_7P, symbol Connector_Generic:Conn_01x07
- added R1, R2, R6: 10k, Resistor_SMD:R_0603_1608Metric, symbol Device:R
- added R10, R11, R14: 100k, Resistor_SMD:R_0603_1608Metric, symbol Device:R
- added R12: 38.3k 1%, Resistor_SMD:R_0603_1608Metric, symbol Device:R
- added R13: 10k 1%, Resistor_SMD:R_0603_1608Metric, symbol Device:R
- added R4, R5: 4.7k, Resistor_SMD:R_0603_1608Metric, symbol Device:R
- added R7: 68R candidate, Resistor_SMD:R_0603_1608Metric, symbol Device:R
- added R8, R9: 5.1k 1%, Resistor_SMD:R_0603_1608Metric, symbol Device:R
- added SW1: RESET, symbol Switch:SW_Push
- added SW2: BOOT, symbol Switch:SW_Push
- added U6: TLV7022DGKR, Package_SO:VSSOP-8_3x3mm_P0.65mm, symbol Comparator:LM2903
Connections:
- net +3V3: now also C3.1, C4.1, C5.1, J4.7 (Pin_7), R1.1, R12.1, R2.1, R4.1, R5.1, R6.1, U6.8 (V+)
- net +5V_LED: now also U4.5 (VCC), C6.1
- net BOOT_GPIO0: now also R2.2, SW2.1
- net CC1: now also R10.1, R8.1
- net CC2: now also R11.1, R9.1
- net EN_RESET: now also C2.1, R1.2, SW1.1
- net GND: now also U4.1, U4.3 (GND), C2.2, C3.2, C4.2, C5.2, C6.2, C7.2, C8.2, C9.2, J4.6 (Pin_6), R13.2, R14.2, R8.2, R9.2, SW1.2, SW2.2, U6.4 (V-)
- net I2C_SCL: now also J4.4 (Pin_4), R5.2
- net I2C_SDA: now also J4.5 (Pin_5), R4.2
- net RGB_DATA_3V3: now also R14.1
- net RGB_DATA_5V: now also U4.4, R7.1
- net RGB_DATA_5V_AFTER_68R: now also R7.2
- net TUSB_INT_N renamed USB_CC_1A5_N
- net USB_CC_1A5_N: now also R6.2, U6.1, U6.7
- new net CC1_FILT: C7.1, R10.2, U6.2 (-)
- new net CC2_FILT: C8.1, R11.2, U6.6 (-)
- new net CC_VREF: C9.1, R12.2, R13.1, U6.3 (+), U6.5 (+)
- no-connect marks 0 -> 3
Other:
- note added: "400kHz pull-ups require measured bus capacitance/rise time."
- note added: "C3/C4 near U1 supply; validate DC bias and rail startup."
- note added: "CC1/CC2: Rd + TLV7022 Rp detector (lower right)"
- note added: "I2C pull-ups (OLED only after TUSB320 removal); R6 = CC detector open-drain pull-up"
- note added: "J4: Rev.A OLED pinout; I2C 0x3C; pins 1-3 open"
- note added: "MCU recovery / decoupling - engineering draft"
- note added: "R7 remains a waveform-validation candidate; C6 near U4."
- note added: "RGB buffer - TI SN74AHCT1G125 Rev.P"
- note added: "RGB data idle bias / OLED module"
- note added: "Switch footprints / passive MPNs remain unselected."
- note added: "U6 uses the LM2903 (LM393) pinout symbol; TLV7022 inputs fault-tolerant to 5.5 V regardless of VCC. C5 = U6 bypass"
- note added: "USB-C sink CC detect: Rd 5.1k 1% per CC; 100k/10n RC rejects PD BMC; TLV7022 open-drain wired-OR"
- note added: "VREF 0.683 V nominal (Type-C vRd 1.5A threshold 0.66 V, biased toward safe Default). USB_CC_1A5_N low = Rp >= 1.5 A"
- note removed: "U2 fixed UFP: PORT=L, ADDR=L (0x60), EN_N=L, VBUS_DET via 900k; no DRP/source control"
